File: hardware/buck_boost.kicad_sch (KiCad schematic)
At the start: 30 parts, among them Q1 IPZ40N04S5L4R8ATMA1, Q2 IPZ40N04S5L4R8ATMA1, U1 TPS55288

Commit message: several updates
Parts:
- removed R9: 7k, Library:R_0603_1608Metric_Pad0.98x0.95mm_HandSolder, symbol Library:R_Small
- added R70: 1k, Library:R_0603_1608Metric_Pad0.98x0.95mm_HandSolder, symbol Library:R_Small
Connections:
- net EN: now also R2.2, R70.1; no longer R2.1
- net GND: now also R70.2; no longer R2.2
- net VIN_24V: now also R2.1
Other:
- note added: "TODO: connect FB/*INT"
- moved on the sheet: R2
Changed lines of the file:
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@@
 		)
 	)
+	(text "TODO: connect FB/*INT"
+		(exclude_from_sim no)
+		(at 214.884 85.09 0)
+		(effects
+			(font
+				(size 1.27 1.27)
+			)
+		)
+	)
 	(text_box "Ripple current (boost): dI_{L,PP} = V_{in}*(V_{out}-V_{in})/(L*f_{sw}*V_{out}) = 20*(22-20)/(4.7u*400k*22) = 970mA\nRipple current (buck): dI_{L,PP} = (V_{in,max} - V_{out})*V_{out} / (L*f_{sw}*V_{in,max}) = (30-15)*15/(4.7u*400k*30) = 4A\nPeak inductr current: I_{L,P} = I_{L,DC} + dI_{L,PP}/2 = 14A\n\n"
 		(exclude_from_sim no)
@@
 	)
 	(symbol
-		(lib_id "Library:R_Small")
-		(at 57.15 63.5 0)
-		(unit 1)
-		(exclude_from_sim no)
-		(in_bom yes)
-		(on_board yes)
-		(dnp no)
-		(fields_autoplaced yes)
-		(property "Reference" "R9"
-			(at 59.69 62.2299 0)
-			(effects
-				(font
-					(size 1.27 1.27)
-				)
-				(justify left)
-			)
-		)
-		(property "Value" "7k"
-			(at 59.69 64.7699 0)
-			(effects
-				(font
-					(size 1.27 1.27)
-				)
-				(justify left)
-			)
-		)
-		(property "Footprint" "Library:R_0603_1608Metric_Pad0.98x0.95mm_HandSolder"
-			(at 57.15 63.5 0)
-			(effects
-				(font
-					(size 1.27 1.27)
-				)
-				(hide yes)
-			)
-		)
-		(property "Datasheet" "~"
-			(at 57.15 63.5 0)
-			(effects
-				(font
-					(size 1.27 1.27)
-				)
-				(hide yes)
-			)
-		)
-		(property "Description" "Resistor, small symbol"
-			(at 57.15 63.5 0)
-			(effects
-				(font
-					(size 1.27 1.27)
-				)
-				(hide yes)
-			)
-		)
-		(property "Digikey-Nr." "311-6.98KHRCT-ND"
-			(at 57.15 63.5 0)
-			(effects
-				(font
-					(size 1.27 1.27)
-				)
-				(hide yes)
-			)
-		)
-		(property "Manufacturer" "YAGEO"
-			(at 57.15 63.5 0)
-			(effects
-				(font
-					(size 1.27 1.27)
-				)
-				(hide yes)
-			)
-		)
-		(property "Manufacturer Nr." "RC0603FR-076K98L"
-			(at 57.15 63.5 0)
-			(effects
-				(font
-					(size 1.27 1.27)
-				)
-				(hide yes)
-			)
-		)
-		(property "Mouser-Nr." "603-RC0603FR-076K98L"
-			(at 57.15 63.5 0)
-			(effects
-				(font
-					(size 1.27 1.27)
-				)
-				(hide yes)
-			)
-		)
-		(property "Manufacturer 2" ""
-			(at 57.15 63.5 0)
-			(effects
-				(font
-					(size 1.27 1.27)
-				)
-				(hide yes)
-			)
-		)
-		(property "Manufacturer-Nr. 2" ""
-			(at 57.15 63.5 0)
-			(effects
-				(font
-					(size 1.27 1.27)
-				)
-				(hide yes)
-			)
-		)
-		(property "Manufacturer-Nr." "RC0603FR-076K98L"
-			(at 57.15 63.5 0)
-			(effects
-				(font
-					(size 1.27 1.27)
-				)
-				(hide yes)
-			)
-		)
-		(pin "1"
-		)
-		(pin "2"
-		)
-		(instances
-			(project "PSB_V1"
-				(path "/1a48cdfa-ddae-48b3-b222-cb19285feeb5/f5092a7f-b2b1-4db8-b72d-823c73afab7a"
-					(reference "R9")
-					(unit 1)
-				)
-			)
-		)
-	)
-	(symbol
 		(lib_id "Library:C_Small")
 		(at 49.53 83.82 0)
@@
 	)
 	(symbol
+		(lib_id "Library:R_Small")
+		(at 57.15 97.79 0)
+		(unit 1)
+		(exclude_from_sim no)
+		(in_bom yes)
+		(on_board yes)
+		(dnp no)
+		(fields_autoplaced yes)
+		(property "Reference" "R70"
+			(at 59.69 96.5199 0)
+			(effects
+				(font
+					(size 1.27 1.27)
+				)
+				(justify left)
+			)
+		)
+		(property "Value" "1k"
+			(at 59.69 99.0599 0)
+			(effects
+				(font
+					(size 1.27 1.27)
+				)
+				(justify left)
+			)
+		)
+		(property "Footprint" "Library:R_0603_1608Metric_Pad0.98x0.95mm_HandSolder"
+			(at 57.15 97.79 0)
+			(effects
+				(font
+					(size 1.27 1.27)
+				)
+				(hide yes)
+			)
+		)
+		(property "Datasheet" "~"
+			(at 57.15 97.79 0)
+			(effects
+				(font
+					(size 1.27 1.27)
+				)
+				(hide yes)
+			)
+		)
+		(property "Description" "Resistor, small symbol"
+			(at 57.15 97.79 0)
+			(effects
+				(font
+					(size 1.27 1.27)
+				)
+				(hide yes)
+			)
+		)
+		(property "Digikey-Nr." "311-1.00KHRCT-ND"
+			(at 57.15 97.79 0)
+			(effects
+				(font
+					(size 1.27 1.27)
+				)
+				(hide yes)
+			)
+		)
+		(property "Manufacturer" "YAGEO"
+			(at 57.15 97.79 0)
+			(effects
+				(font
+					(size 1.27 1.27)
+				)
+				(hide yes)
+			)
+		)
+		(property "Manufacturer Nr." "RC0603FR-071KL"
+			(at 57.15 97.79 0)
+			(effects
+				(font
+					(size 1.27 1.27)
+				)
+				(hide yes)
+			)
+		)
+		(property "Mouser-Nr." "603-RC0603FR-071KL"
+			(at 57.15 97.79 0)
+			(effects
+				(font
+					(size 1.27 1.27)
+				)
+				(hide yes)
+			)
+		)
+		(property "Manufacturer 2" ""
+			(at 57.15 97.79 0)
+			(effects
+				(font
+					(size 1.27 1.27)
+				)
+				(hide yes)
+			)
+		)
+		(property "Manufacturer-Nr. 2" ""
+			(at 57.15 97.79 0)
+			(effects
+				(font
+					(size 1.27 1.27)
+				)
+				(hide yes)
+			)
+		)
+		(property "Manufacturer-Nr." "RC0603FR-071KL"
+			(at 57.15 97.79 0)
+			(effects
+				(font
+					(size 1.27 1.27)
+				)
+				(hide yes)
+			)
+		)
+		(pin "1"
+		)
+		(pin "2"
+		)
+		(instances
+			(project "PowerSupplyModule"
+				(path "/1a48cdfa-ddae-48b3-b222-cb19285feeb5/f5092a7f-b2b1-4db8-b72d-823c73afab7a"
+					(reference "R70")
+					(unit 1)
+				)
+			)
+		)
+	)
+	(symbol
 		(lib_id "Library:C_Small")
 		(at 267.97 71.12 90)
@@
 	(symbol
 		(lib_id "Library:R_Small")
-		(at 57.15 97.79 0)
+		(at 57.15 63.5 0)
 		(unit 1)
 		(exclude_from_sim no)
@@
 		(fields_autoplaced yes)
 		(property "Reference" "R2"
-			(at 59.69 96.5199 0)
+			(at 59.69 62.2299 0)
 			(effects
 				(font
@@
 		)
 		(property "Value" "10k"
-			(at 59.69 99.0599 0)
+			(at 59.69 64.7699 0)
 			(effects
 				(font
@@
 		)
 		(property "Footprint" "Library:R_0603_1608Metric_Pad0.98x0.95mm_HandSolder"
-			(at 57.15 97.79 0)
+			(at 57.15 63.5 0)
 			(effects
 				(font
@@
 		)
 		(property "Datasheet" "~"
-			(at 57.15 97.79 0)
+			(at 57.15 63.5 0)
 			(effects
 				(font
@@
 		)
 		(property "Description" "Resistor, small symbol"
-			(at 57.15 97.79 0)
+			(at 57.15 63.5 0)
 			(effects
 				(font
@@
 		)
 		(property "Digikey-Nr." "311-10.0KHRCT-ND"
-			(at 57.15 97.79 0)
+			(at 57.15 63.5 0)
 			(effects
 				(font
@@
 		)
 		(property "Manufacturer" "YAGEO"
-			(at 57.15 97.79 0)
+			(at 57.15 63.5 0)
 			(effects
 				(font
@@
 		)
 		(property "Manufacturer Nr." "RC0603FR-0710KL"
-			(at 57.15 97.79 0)
+			(at 57.15 63.5 0)
 			(effects
 				(font
@@
 		)
 		(property "Mouser-Nr." "603-RC0603FR-0710KL"
-			(at 57.15 97.79 0)
+			(at 57.15 63.5 0)
 			(effects
 				(font
@@
 		)
 		(property "Manufacturer 2" ""
-			(at 57.15 97.79 0)
+			(at 57.15 63.5 0)
 			(effects
 				(font
@@
 		)
 		(property "Manufacturer-Nr. 2" ""
-			(at 57.15 97.79 0)
+			(at 57.15 63.5 0)
 			(effects
 				(font
@@
 		)
 		(property "Manufacturer-Nr." "RC0603FR-0710KL"
-			(at 57.15 97.79 0)
+			(at 57.15 63.5 0)
 			(effects
 				(font
